File: Qwiic_4_Pin_Fan_Controller.brd (EAGLE design)
At the start: 45.7 x 25.4 mm, 74 parts, among them J1 QWIIC_RIGHT_ANGLE, J2 QWIIC_RIGHT_ANGLE, J3 AVR_SPI_PROG_3X2TESTPOINTS, Q1 20V/4.2A/52mΩ/1.4W, Q2 310mA/60V/1.6Ω, Q3 310mA/60V/1.6Ω, Q7 20V/4.2A/52mΩ/1.4W, U1 ATtiny841, U3 PAM2401, Y2 16MHz

Commit message: x02 silk change and gerbers
-Fix a silk label on the bottom
-Panelize and CAM Production Files
Parts:
- added U$31: (no value), output:#FAN_VCC_#0
- added U$32: (no value), output:_#_20VDC0
Changed lines of the file:
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@@
 <attribute name="VALUE" x="20.955" y="18.415" size="0.6096" layer="27" font="vector" ratio="20" rot="R180" align="top-center"/>
 </element>
+<element name="U$31" library="output" package="#FAN_VCC_#0" value="" x="24.13" y="23.622" smashed="yes" rot="MR90"/>
+<element name="U$32" library="output" package="_#_20VDC0" value="" x="22.86" y="22.86" smashed="yes" rot="MR90"/>
 </elements>
 <signals>
@@
 <wire x1="6.731" y1="12.7" x2="21.59" y2="12.7" width="0.508" layer="16"/>
 <via x="38.1" y="12.192" extent="1-16" drill="0.3"/>
-<wire x1="21.59" y1="12.7" x2="27.94" y2="12.7" width="0.508" layer="16"/>
-<wire x1="27.94" y1="12.7" x2="30.861" y2="12.7" width="0.508" layer="16"/>
+<wire x1="21.59" y1="12.7" x2="30.861" y2="12.7" width="0.508" layer="16"/>
 <wire x1="30.861" y1="12.7" x2="31.496" y2="12.7" width="0.508" layer="16"/>
 <wire x1="38.1" y1="12.192" x2="32.004" y2="12.192" width="0.508" layer="16"/>
