File: Production/Qwiic_4_Pin_Fan_Controller-Panel.brd (EAGLE design)
At the start: 158.2 x 143.3 mm, 1116 parts, among them J1 QWIIC_RIGHT_ANGLE, J13 QWIIC_RIGHT_ANGLE, J14 QWIIC_RIGHT_ANGLE, J15 AVR_SPI_PROG_3X2TESTPOINTS, J19 QWIIC_RIGHT_ANGLE, J2 QWIIC_RIGHT_ANGLE, J20 QWIIC_RIGHT_ANGLE, J21 AVR_SPI_PROG_3X2TESTPOINTS, J25 QWIIC_RIGHT_ANGLE, J26 QWIIC_RIGHT_ANGLE, J27 AVR_SPI_PROG_3X2TESTPOINTS, J3 AVR_SPI_PROG_3X2TESTPOINTS, J31 QWIIC_RIGHT_ANGLE, J32 QWIIC_RIGHT_ANGLE, J33 AVR_SPI_PROG_3X2TESTPOINTS, J37 QWIIC_RIGHT_ANGLE, J38 QWIIC_RIGHT_ANGLE, J39 AVR_SPI_PROG_3X2TESTPOINTS, J43 QWIIC_RIGHT_ANGLE, J44 QWIIC_RIGHT_ANGLE, J45 AVR_SPI_PROG_3X2TESTPOINTS, J49 QWIIC_RIGHT_ANGLE, J50 QWIIC_RIGHT_ANGLE, J51 AVR_SPI_PROG_3X2TESTPOINTS, J55 QWIIC_RIGHT_ANGLE, J56 QWIIC_RIGHT_ANGLE, J57 AVR_SPI_PROG_3X2TESTPOINTS, J61 QWIIC_RIGHT_ANGLE, J62 QWIIC_RIGHT_ANGLE, J63 AVR_SPI_PROG_3X2TESTPOINTS, J67 QWIIC_RIGHT_ANGLE, J68 QWIIC_RIGHT_ANGLE, J69 AVR_SPI_PROG_3X2TESTPOINTS, J7 QWIIC_RIGHT_ANGLE, J73 QWIIC_RIGHT_ANGLE, J74 QWIIC_RIGHT_ANGLE, J75 AVR_SPI_PROG_3X2TESTPOINTS, J79 QWIIC_RIGHT_ANGLE, J8 QWIIC_RIGHT_ANGLE, J80 QWIIC_RIGHT_ANGLE, J81 AVR_SPI_PROG_3X2TESTPOINTS, J85 QWIIC_RIGHT_ANGLE, J86 QWIIC_RIGHT_ANGLE, J87 AVR_SPI_PROG_3X2TESTPOINTS, J9 AVR_SPI_PROG_3X2TESTPOINTS, Q1 20V/4.2A/52mΩ/1.4W, Q10 310mA/60V/1.6Ω, Q11 310mA/60V/1.6Ω, Q12 20V/4.2A/52mΩ/1.4W, Q13 310mA/60V/1.6Ω, Q14 310mA/60V/1.6Ω, Q15 20V/4.2A/52mΩ/1.4W, Q16 310mA/60V/1.6Ω, Q17 310mA/60V/1.6Ω, Q18 20V/4.2A/52mΩ/1.4W, Q19 310mA/60V/1.6Ω, Q2 310mA/60V/1.6Ω, Q20 310mA/60V/1.6Ω, Q21 20V/4.2A/52mΩ/1.4W, Q22 310mA/60V/1.6Ω, Q23 310mA/60V/1.6Ω, Q24 20V/4.2A/52mΩ/1.4W, Q25 310mA/60V/1.6Ω, Q26 310mA/60V/1.6Ω, Q27 20V/4.2A/52mΩ/1.4W, Q28 310mA/60V/1.6Ω, Q29 310mA/60V/1.6Ω, Q3 310mA/60V/1.6Ω, Q30 20V/4.2A/52mΩ/1.4W, Q31 310mA/60V/1.6Ω, Q32 310mA/60V/1.6Ω, Q33 20V/4.2A/52mΩ/1.4W, Q34 310mA/60V/1.6Ω, Q35 310mA/60V/1.6Ω, Q36 20V/4.2A/52mΩ/1.4W, Q37 310mA/60V/1.6Ω, Q38 310mA/60V/1.6Ω, Q39 20V/4.2A/52mΩ/1.4W, Q4 310mA/60V/1.6Ω, Q40 310mA/60V/1.6Ω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

Commit message: x02 silk change and gerbers
-Fix a silk label on the bottom
-Panelize and CAM Production Files
Parts:
- removed C41, C44, C46, C49, C51, C54, C56, C59, C61, C64, C66, C69, C71, C74: 22pF, SparkFun-Capacitors:0603
- removed C42, C47, C52, C57, C62, C67, C72: 10uF, SparkFun-Capacitors:0603
- removed C43, C48, C53, C58, C63, C68, C73: 0.1uF, SparkFun-Capacitors:0603
- removed C45, C50, C55, C60, C65, C70, C75: 22uF, SparkFun-Capacitors:0805
- removed D25, D26, D28, D29, D31, D32, D34, D35, D37, D38, D40, D41, D43, D44: 3.6V, SparkFun-DiscreteSemi:SOD-323
- removed D27, D30, D33, D36, D39, D42, D45: RED, SparkFun-LED:LED-0603
- removed F10, F11, F12, F13, F14, F15, F9: 6V/0.75A, SparkFun-Fuses:1206
- removed J49, J50, J55, J56, J61, J62, J67, J68, J73, J74, J79, J80, J85, J86: QWIIC_RIGHT_ANGLE, SparkFun-Connectors:JST04_1MM_RA
- removed J51, J57, J63, J69, J75, J81, J87: AVR_SPI_PROG_3X2TESTPOINTS, SparkFun-Connectors:2X3_TEST_POINTS
- removed J52, J53, J58, J59, J64, J65, J70, J71, J76, J77, J82, J83, J88, J89: (no value), SparkFun-Connectors:1X04_NO_SILK
- removed J54, J60, J66, J72, J78, J84, J90: (no value), SparkFun-Connectors:1X02_NO_SILK
- removed JP1, JP10, JP11, JP12, JP13, JP14, JP15, JP2, JP3, JP4, JP5, JP6, JP7, JP8, JP9: JUMPER-SMT_2_NC_TRACE_NO-SILK, SparkFun-Jumpers:SMT-JUMPER_2_NC_TRACE_NO-SILK
- removed L10, L11, L12, L13, L14, L15, L9: 2.2μH, SparkFun-Coils:0806
- removed Q41, Q43, Q44: 310mA/60V/1.6Ω, SparkFun-DiscreteSemi:SOT323
- removed Q42, Q45: 20V/4.2A/52mΩ/1.4W, SparkFun-DiscreteSemi:SOT23-3
- removed R105, R106, R112, R113, R116, R117, R123, R124, R127, R128, R134, R135, R138, R139, R145, R146, R149, R150, R156, R157, R160, R161: 2.2k, SparkFun-Resistors:0603
- removed R107, R110, R118, R121, R129, R132, R140, R143, R151, R154, R162, R165: 1k, SparkFun-Resistors:0603
- removed R108, R109, R114, R119, R120, R125, R130, R131, R136, R141, R142, R147, R152, R153, R158, R163, R164: 10k, SparkFun-Resistors:0603
- removed R111, R122, R133, R144, R155: 750K, SparkFun-Resistors:0603
- removed R115, R126, R137, R148, R159: 100k, SparkFun-Resistors:0603
- removed U$289, U$327, U$365, U$403, U$441, U$479, U$517, U$555: (no value), output:#_SDA#0
- removed U$290, U$328, U$366, U$404, U$442, U$480, U$518, U$556: (no value), output:#_SCL#0
- removed U$291, U$297, U$329, U$335, U$367, U$373, U$405, U$411, U$443, U$449, U$481, U$487, U$519, U$525, U$557, U$563: (no value), output:QWIIC_PC_FAN_CONTROLLER0
- removed U$292, U$330, U$368, U$406, U$444, U$482, U$520, U$558: (no value), output:CUT_JUMPER_BEFORE0
- removed U$293, U$331, U$369, U$407, U$445, U$483, U$521, U$559: (no value), output:SUPPLYING_UP_TO0
- removed U$294, U$332, U$370, U$408, U$446, U$484, U$522, U$560: (no value), output:12VDC_EXTERNAL0
- removed U$295, U$333, U$371, U$409, U$447, U$485, U$523, U$561: (no value), output:FAN_POWER_SUPPLY0
- removed U$296, U$319, U$334, U$357, U$372, U$395, U$410, U$433, U$448, U$471, U$486, U$509, U$524, U$547, U$562: (no value), SparkX:SPARKX-SMALL
- removed U$298, U$336, U$374, U$412, U$450, U$488, U$526, U$564: (no value), SparkFun-Aesthetics:OSHW-LOGO-S
- removed U$299, U$337, U$375, U$413, U$451, U$489, U$527, U$565: (no value), output:#_FAN_VCC#0
- removed U$300, U$338, U$376, U$414, U$452, U$490, U$528, U$566: (no value), output:#PID_TUNING0
- removed U$301, U$339, U$377, U$415, U$453, U$491, U$529, U$567: (no value), output:KI0
- removed U$302, U$340, U$378, U$416, U$454, U$492, U$530, U$568: (no value), output:KP0
- removed U$303, U$341, U$379, U$417, U$455, U$493, U$531, U$569: (no value), output:PWR0
- removed U$304, U$342, U$380, U$418, U$456, U$494, U$532, U$570: (no value), turn_indicators:TURN_INDICATOR#SVG0
- removed U$305, U$306, U$307, U$308, U$343, U$344, U$345, U$346, U$381, U$382, U$383, U$384, U$419, U$420, U$421, U$422, U$457, U$458, U$459, U$460, U$495, U$496, U$497, U$498, U$533, U$534, U$535, U$536: (no value), SparkFun-Hardware:STAND-OFF
- removed U$309, U$313, U$321, U$347, U$351, U$359, U$385, U$389, U$397, U$423, U$427, U$435, U$461, U$465, U$473, U$499, U$503, U$511, U$537, U$541, U$549: (no value), output:#_GND#0
- removed U$310, U$348, U$386, U$424, U$462, U$500, U$538: (no value), output:#_VCC#0
- removed U$311, U$349, U$387, U$425, U$463, U$501, U$539: (no value), output:#_TACH#0
- removed U$312, U$350, U$388, U$426, U$464, U$502, U$540: (no value), output:#_PWM#0
- removed U$314, U$320, U$325, U$352, U$358, U$363, U$390, U$396, U$401, U$428, U$434, U$439, U$466, U$472, U$477, U$504, U$510, U$515, U$542, U$548, U$553: (no value), output:#GND_#0
- removed U$315, U$353, U$391, U$429, U$467, U$505, U$543: (no value), output:#3#3V_#0
- removed U$316, U$354, U$392, U$430, U$468, U$506, U$544: (no value), output:#SDA_#0
- removed U$317, U$355, U$393, U$431, U$469, U$507, U$545: (no value), output:#SCL_#0
- removed U$318, U$356, U$394, U$432, U$470, U$508, U$546: (no value), SparkFun-Aesthetics:QWIIC_3MM
- removed U$322, U$360, U$398, U$436, U$474, U$512, U$550: (no value), output:#VCC_#0
- removed U$323, U$361, U$399, U$437, U$475, U$513, U$551: (no value), output:#TACH_#0
- removed U$324, U$362, U$400, U$438, U$476, U$514, U$552: (no value), output:#PWM_#0
- removed U$326, U$364, U$402, U$440, U$478, U$516, U$554: (no value), output:#_3#3V#0
- removed U17, U19, U21, U23, U25, U27, U29: ATtiny841, SparkFun-IC-Microcontroller:SO14
- removed U18, U20, U22, U24, U26, U28, U30: PAM2401, SparkFun-IC-Power:MSOP8
- removed VR17, VR18, VR19, VR20, VR21, VR22, VR23, VR24, VR25, VR26, VR27, VR28, VR29, VR30: 10k, SparkFun-Resistors:TRIMPOT-SMD-3MM-CLOSED
- removed Y10, Y11, Y12, Y13, Y14, Y15, Y9: 16MHz, SparkFun-Clocks:CRYSTAL-SMD-2.0X1.6MM
- Q10, Q20, Q25, Q35, Q40, Q8: value 310mA/60V/1.6Ω -> (none); device SparkFun-DiscreteSemi:SOT323 -> SparkFun-DiscreteSemi:SOT363_PHILIPS
- Q12, Q21, Q27, Q36: value 20V/4.2A/52mΩ/1.4W -> 310mA/60V/1.6Ω; device SparkFun-DiscreteSemi:SOT23-3 -> SparkFun-DiscreteSemi:SOT323
- Q13, Q14, Q19, Q23, Q28, Q29, Q34, Q38, Q7: value 310mA/60V/1.6Ω -> 20V/4.2A/52mΩ/1.4W; device SparkFun-DiscreteSemi:SOT323 -> SparkFun-DiscreteSemi:SOT23-3
- Q15, Q30: value 20V/4.2A/52mΩ/1.4W -> (none); device SparkFun-DiscreteSemi:SOT23-3 -> SparkFun-DiscreteSemi:SOT363_PHILIPS
- R10: value 750K -> 47k; device SparkFun-Resistors:0603 -> SparkFun-Resistors:0603@1
- R100, R23, R56, R78: value 750K -> 10k; device SparkFun-Resistors:0603 -> SparkFun-Resistors:0603@1
- R101, R12, R17, R35, R36, R39, R61, R62, R69, R91, R95: value 2.2k -> 10k; device SparkFun-Resistors:0603 -> SparkFun-Resistors:0603@1
- R102, R24, R47, R50, R73: value 2.2k -> 1k
- R103, R64: value 10k -> 47k; device SparkFun-Resistors:0603 -> SparkFun-Resistors:0603@1
- R104, R49, R82: value 100k -> 10k; device SparkFun-Resistors:0603 -> SparkFun-Resistors:0603@1
- R14, R40, R79: value 2.2k -> 750K
- R15, R20, R32, R42, R54, R59, R81, R97, R98: value 10k -> 2.2k
- R16, R71, R93: value 100k -> 2.2k
- R18, R57, R83: value 2.2k -> 100k
- R19, R33, R41, R55, R85: value 1k -> 2.2k
- R2, R26, R43, R48, R65, R7, R75, R8, R87: device SparkFun-Resistors:0603 -> SparkFun-Resistors:0603@1
- R21, R37, R76, R86: value 10k -> 1k
- R22, R30, R52, R74, R88: value 1k -> 10k; device SparkFun-Resistors:0603 -> SparkFun-Resistors:0603@1
- R25, R51, R90: value 2.2k -> 47k; device SparkFun-Resistors:0603 -> SparkFun-Resistors:0603@1
- R27: value 100k -> 750K
- R31, R70: value 10k -> 100k
- R34, R89: value 750K -> 1k
- R38: value 100k -> 47k; device SparkFun-Resistors:0603 -> SparkFun-Resistors:0603@1
- R44, R96: value 1k -> 100k
- R45, R67: value 750K -> 2.2k
- R53, R92: value 10k -> 750K
- R60: value 100k -> 1k
- R66: value 1k -> 750K
- R77: value 1k -> 47k; device SparkFun-Resistors:0603 -> SparkFun-Resistors:0603@1
- U$100: device output:#_SCL#0 -> SparkFun-Aesthetics:OSHW-LOGO-S
- U$101: device output:QWIIC_PC_FAN_CONTROLLER0 -> output:#_FAN_VCC#0
- U$102: device output:CUT_JUMPER_BEFORE0 -> output:#PID_TUNING0
- U$103: device output:SUPPLYING_UP_TO0 -> output:KI0
- U$104: device output:12VDC_EXTERNAL0 -> output:KP0
- U$105: device output:FAN_POWER_SUPPLY0 -> output:PWR0
- U$106: device SparkX:SPARKX-SMALL -> turn_indicators:TURN_INDICATOR#SVG0
- U$107, U$215: device output:QWIIC_PC_FAN_CONTROLLER0 -> output:#FAN_VCC_#0
- U$108: device SparkFun-Aesthetics:OSHW-LOGO-S -> output:_#_20VDC0
- U$109, U$147: device output:#_FAN_VCC#0 -> SparkFun-Hardware:STAND-OFF
- U$110, U$148: device output:#PID_TUNING0 -> SparkFun-Hardware:STAND-OFF
- U$111, U$73: device output:KI0 -> SparkFun-Hardware:STAND-OFF
- U$112, U$74: device output:KP0 -> SparkFun-Hardware:STAND-OFF
- U$113, U$189: device output:PWR0 -> output:#_GND#0
- U$114: device turn_indicators:TURN_INDICATOR#SVG0 -> output:#_VCC#0
- U$115, U$79: device SparkFun-Hardware:STAND-OFF -> output:#_TACH#0
- U$116, U$80: device SparkFun-Hardware:STAND-OFF -> output:#_PWM#0
- U$117, U$153, U$269, U$41, U$77: device SparkFun-Hardware:STAND-OFF -> output:#_GND#0
- U$118, U$154, U$232, U$268: device SparkFun-Hardware:STAND-OFF -> output:#GND_#0
- U$119, U$47: device output:#_GND#0 -> output:#3#3V_#0
- U$120: device output:#_VCC#0 -> output:#SDA_#0
- U$121: device output:#_TACH#0 -> output:#SCL_#0
- U$122: device output:#_PWM#0 -> SparkFun-Aesthetics:QWIIC_3MM
- U$123, U$195: device output:#_GND#0 -> SparkX:SPARKX-SMALL
- U$125: device output:#3#3V_#0 -> output:#_GND#0
- U$126: device output:#SDA_#0 -> output:#VCC_#0
- U$127: device output:#SCL_#0 -> output:#TACH_#0
- U$128: device SparkFun-Aesthetics:QWIIC_3MM -> output:#PWM_#0
- U$129: device SparkX:SPARKX-SMALL -> output:#GND_#0
- U$130, U$238: device output:#GND_#0 -> output:#_3#3V#0
- U$131, U$275: device output:#_GND#0 -> output:#_SDA#0
- U$132: device output:#VCC_#0 -> output:#_SCL#0
- U$133, U$171: device output:#TACH_#0 -> output:QWIIC_PC_FAN_CONTROLLER0
- U$134: device output:#PWM_#0 -> SparkX:SPARKX-SMALL
- U$135, U$97: device output:#GND_#0 -> output:QWIIC_PC_FAN_CONTROLLER0
- U$136: device output:#_3#3V#0 -> SparkFun-Aesthetics:OSHW-LOGO-S
- U$137: device output:#_SDA#0 -> output:#_FAN_VCC#0
- U$138: device output:#_SCL#0 -> output:#PID_TUNING0
- U$139: device output:QWIIC_PC_FAN_CONTROLLER0 -> output:KI0
- U$140: device output:CUT_JUMPER_BEFORE0 -> output:KP0
- U$141: device output:SUPPLYING_UP_TO0 -> output:PWR0
- U$142: device output:12VDC_EXTERNAL0 -> turn_indicators:TURN_INDICATOR#SVG0
- U$143: device output:FAN_POWER_SUPPLY0 -> output:#FAN_VCC_#0
- U$144: device SparkX:SPARKX-SMALL -> output:_#_20VDC0
- U$145, U$183, U$253: device output:QWIIC_PC_FAN_CONTROLLER0 -> SparkFun-Hardware:STAND-OFF
- U$146, U$184: device SparkFun-Aesthetics:OSHW-LOGO-S -> SparkFun-Hardware:STAND-OFF
- U$149, U$225: device output:KI0 -> output:#_GND#0
- U$150: device output:KP0 -> output:#_VCC#0
- U$151: device output:PWR0 -> output:#_TACH#0
- U$152: device turn_indicators:TURN_INDICATOR#SVG0 -> output:#_PWM#0
- U$155, U$191: device SparkFun-Hardware:STAND-OFF -> output:#3#3V_#0
- U$156, U$192: device SparkFun-Hardware:STAND-OFF -> output:#SDA_#0
- U$157, U$85: device output:#_GND#0 -> output:#SCL_#0
- U$158: device output:#_VCC#0 -> SparkFun-Aesthetics:QWIIC_3MM
- U$159: device output:#_TACH#0 -> SparkX:SPARKX-SMALL
- U$160, U$46: device output:#_PWM#0 -> output:#GND_#0
- U$162, U$54: device output:#GND_#0 -> output:#VCC_#0
- U$163: device output:#3#3V_#0 -> output:#TACH_#0
- U$164: device output:#SDA_#0 -> output:#PWM_#0
- U$165: device output:#SCL_#0 -> output:#GND_#0
- U$166: device SparkFun-Aesthetics:QWIIC_3MM -> output:#_3#3V#0
- U$167: device SparkX:SPARKX-SMALL -> output:#_SDA#0
- U$168, U$276: device output:#GND_#0 -> output:#_SCL#0
- U$169, U$207: device output:#_GND#0 -> output:QWIIC_PC_FAN_CONTROLLER0
- U$170: device output:#VCC_#0 -> SparkX:SPARKX-SMALL
- U$172: device output:#PWM_#0 -> SparkFun-Aesthetics:OSHW-LOGO-S
- U$173: device output:#GND_#0 -> output:#_FAN_VCC#0
- U$174: device output:#_3#3V#0 -> output:#PID_TUNING0
- U$175: device output:#_SDA#0 -> output:KI0
- U$176: device output:#_SCL#0 -> output:KP0
- U$177, U$69: device output:QWIIC_PC_FAN_CONTROLLER0 -> output:PWR0
- U$178: device output:CUT_JUMPER_BEFORE0 -> turn_indicators:TURN_INDICATOR#SVG0
- U$179: device output:SUPPLYING_UP_TO0 -> output:#FAN_VCC_#0
- U$180: device output:12VDC_EXTERNAL0 -> output:_#_20VDC0
- U$181, U$219, U$34: device output:FAN_POWER_SUPPLY0 -> SparkFun-Hardware:STAND-OFF
- U$182, U$220: device SparkX:SPARKX-SMALL -> SparkFun-Hardware:STAND-OFF
- U$185, U$261: device output:#_FAN_VCC#0 -> output:#_GND#0
- U$186: device output:#PID_TUNING0 -> output:#_VCC#0
- U$187: device output:KI0 -> output:#_TACH#0
- U$188: device output:KP0 -> output:#_PWM#0
- U$190: device turn_indicators:TURN_INDICATOR#SVG0 -> output:#GND_#0
- U$193, U$229: device SparkFun-Hardware:STAND-OFF -> output:#SCL_#0
- U$194, U$230: device SparkFun-Hardware:STAND-OFF -> SparkFun-Aesthetics:QWIIC_3MM
- U$196, U$82: device output:#_VCC#0 -> output:#GND_#0
- U$197, U$45: device output:#_TACH#0 -> output:#_GND#0
- U$198: device output:#_PWM#0 -> output:#VCC_#0
- U$199, U$271, U$55: device output:#_GND#0 -> output:#TACH_#0
- U$200, U$92: device output:#GND_#0 -> output:#PWM_#0
- U$201: device output:#3#3V_#0 -> output:#GND_#0
- U$202: device output:#SDA_#0 -> output:#_3#3V#0
- U$203: device output:#SCL_#0 -> output:#_SDA#0
- U$204: device SparkFun-Aesthetics:QWIIC_3MM -> output:#_SCL#0
- U$205, U$243: device SparkX:SPARKX-SMALL -> output:QWIIC_PC_FAN_CONTROLLER0
- U$206: device output:#GND_#0 -> SparkX:SPARKX-SMALL
- U$208: device output:#VCC_#0 -> SparkFun-Aesthetics:OSHW-LOGO-S
- U$209: device output:#TACH_#0 -> output:#_FAN_VCC#0
- U$210: device output:#PWM_#0 -> output:#PID_TUNING0
- U$211: device output:#GND_#0 -> output:KI0
- U$212: device output:#_3#3V#0 -> output:KP0
- U$213: device output:#_SDA#0 -> output:PWR0
- U$214: device output:#_SCL#0 -> turn_indicators:TURN_INDICATOR#SVG0
- U$216: device output:CUT_JUMPER_BEFORE0 -> output:_#_20VDC0
- U$217, U$255: device output:SUPPLYING_UP_TO0 -> SparkFun-Hardware:STAND-OFF
- U$218, U$256, U$33: device output:12VDC_EXTERNAL0 -> SparkFun-Hardware:STAND-OFF
- U$221: device output:QWIIC_PC_FAN_CONTROLLER0 -> output:#_GND#0
- U$222: device SparkFun-Aesthetics:OSHW-LOGO-S -> output:#_VCC#0
- U$223: device output:#_FAN_VCC#0 -> output:#_TACH#0
- U$224: device output:#PID_TUNING0 -> output:#_PWM#0
- U$226: device output:KP0 -> output:#GND_#0
- U$227: device output:PWR0 -> output:#3#3V_#0
- U$228: device turn_indicators:TURN_INDICATOR#SVG0 -> output:#SDA_#0
- U$231, U$267: device SparkFun-Hardware:STAND-OFF -> SparkX:SPARKX-SMALL
- U$234: device output:#_VCC#0 -> output:#VCC_#0
- U$235: device output:#_TACH#0 -> output:#TACH_#0
- U$236: device output:#_PWM#0 -> output:#PWM_#0
- U$237, U$93: device output:#_GND#0 -> output:#GND_#0
- U$239: device output:#3#3V_#0 -> output:#_SDA#0
- U$240: device output:#SDA_#0 -> output:#_SCL#0
- U$241, U$279: device output:#SCL_#0 -> output:QWIIC_PC_FAN_CONTROLLER0
- U$242: device SparkFun-Aesthetics:QWIIC_3MM -> SparkX:SPARKX-SMALL
- U$244: device output:#GND_#0 -> SparkFun-Aesthetics:OSHW-LOGO-S
- U$245: device output:#_GND#0 -> output:#_FAN_VCC#0
- U$246: device output:#VCC_#0 -> output:#PID_TUNING0
- U$247: device output:#TACH_#0 -> output:KI0
- U$248: device output:#PWM_#0 -> output:KP0
- U$249: device output:#GND_#0 -> output:PWR0
- U$250: device output:#_3#3V#0 -> turn_indicators:TURN_INDICATOR#SVG0
- U$251: device output:#_SDA#0 -> output:#FAN_VCC_#0
- U$252: device output:#_SCL#0 -> output:_#_20VDC0
- U$254: device output:CUT_JUMPER_BEFORE0 -> SparkFun-Hardware:STAND-OFF
- U$257: device output:FAN_POWER_SUPPLY0 -> output:#_GND#0
- U$258: device SparkX:SPARKX-SMALL -> output:#_VCC#0
- U$259: device output:QWIIC_PC_FAN_CONTROLLER0 -> output:#_TACH#0
- U$260: device SparkFun-Aesthetics:OSHW-LOGO-S -> output:#_PWM#0
- U$262: device output:#PID_TUNING0 -> output:#GND_#0
- U$263: device output:KI0 -> output:#3#3V_#0
- U$264: device output:KP0 -> output:#SDA_#0
- U$265: device output:PWR0 -> output:#SCL_#0
- U$266: device turn_indicators:TURN_INDICATOR#SVG0 -> SparkFun-Aesthetics:QWIIC_3MM
- U$270: device SparkFun-Hardware:STAND-OFF -> output:#VCC_#0
- U$272: device output:#_VCC#0 -> output:#PWM_#0
- U$273: device output:#_TACH#0 -> output:#GND_#0
- U$274: device output:#_PWM#0 -> output:#_3#3V#0
- U$277: device output:#3#3V_#0 -> output:QWIIC_PC_FAN_CONTROLLER0
- U$278: device output:#SDA_#0 -> SparkX:SPARKX-SMALL
- U$280: device SparkFun-Aesthetics:QWIIC_3MM -> SparkFun-Aesthetics:OSHW-LOGO-S
- U$281: device SparkX:SPARKX-SMALL -> output:#_FAN_VCC#0
- U$282: device output:#GND_#0 -> output:#PID_TUNING0
- U$283: device output:#_GND#0 -> output:KI0
- U$284: device output:#VCC_#0 -> output:KP0
- U$285: device output:#TACH_#0 -> output:PWR0
- U$286: device output:#PWM_#0 -> turn_indicators:TURN_INDICATOR#SVG0
- U$287: device output:#GND_#0 -> output:#FAN_VCC_#0
- U$288: device output:#_3#3V#0 -> output:_#_20VDC0
- U$31: device output:CUT_JUMPER_BEFORE0 -> output:#FAN_VCC_#0
- U$32: device output:SUPPLYING_UP_TO0 -> output:_#_20VDC0
- U$42, U$78: device SparkFun-Hardware:STAND-OFF -> output:#_VCC#0
- U$43: device output:#_GND#0 -> output:#_TACH#0
- U$44: device output:#_VCC#0 -> output:#_PWM#0
- U$48: device output:#GND_#0 -> output:#SDA_#0
- U$49: device output:#3#3V_#0 -> output:#SCL_#0
- U$50: device output:#SDA_#0 -> SparkFun-Aesthetics:QWIIC_3MM
- U$51: device output:#SCL_#0 -> SparkX:SPARKX-SMALL
- U$52: device SparkFun-Aesthetics:QWIIC_3MM -> output:#GND_#0
- U$53: device SparkX:SPARKX-SMALL -> output:#_GND#0
- U$56: device output:#VCC_#0 -> output:#PWM_#0
- U$57: device output:#TACH_#0 -> output:#GND_#0
- U$58: device output:#PWM_#0 -> output:#_3#3V#0
- U$59: device output:#GND_#0 -> output:#_SDA#0
- U$60: device output:#_3#3V#0 -> output:#_SCL#0
- U$61, U$99: device output:#_SDA#0 -> output:QWIIC_PC_FAN_CONTROLLER0
- U$62: device output:#_SCL#0 -> SparkX:SPARKX-SMALL
- U$64: device output:CUT_JUMPER_BEFORE0 -> SparkFun-Aesthetics:OSHW-LOGO-S
- U$65: device output:SUPPLYING_UP_TO0 -> output:#_FAN_VCC#0
- U$66: device output:12VDC_EXTERNAL0 -> output:#PID_TUNING0
- U$67: device output:FAN_POWER_SUPPLY0 -> output:KI0
- U$68: device SparkX:SPARKX-SMALL -> output:KP0
- U$70: device SparkFun-Aesthetics:OSHW-LOGO-S -> turn_indicators:TURN_INDICATOR#SVG0
- U$71: device output:#_FAN_VCC#0 -> output:#FAN_VCC_#0
- U$72: device output:#PID_TUNING0 -> output:_#_20VDC0
- U$75: device output:PWR0 -> SparkFun-Hardware:STAND-OFF
- U$76: device turn_indicators:TURN_INDICATOR#SVG0 -> SparkFun-Hardware:STAND-OFF
- U$83: device output:#_TACH#0 -> output:#3#3V_#0
- U$84: device output:#_PWM#0 -> output:#SDA_#0
- U$86: device output:#GND_#0 -> SparkFun-Aesthetics:QWIIC_3MM
- U$87: device output:#3#3V_#0 -> SparkX:SPARKX-SMALL
- U$88: device output:#SDA_#0 -> output:#GND_#0
- U$89: device output:#SCL_#0 -> output:#_GND#0
- U$90: device SparkFun-Aesthetics:QWIIC_3MM -> output:#VCC_#0
- U$91: device SparkX:SPARKX-SMALL -> output:#TACH_#0
- U$94: device output:#VCC_#0 -> output:#_3#3V#0
- U$95: device output:#TACH_#0 -> output:#_SDA#0
- U$96: device output:#PWM_#0 -> output:#_SCL#0
- U$98: device output:#_3#3V#0 -> SparkX:SPARKX-SMALL
- moved U$217 129.0 mm to (2.54, 100.6), flipped to the top, turned to 0 degrees
- moved R89 125.9 mm to (2.54, 94.9), turned to 180 degrees
- moved R63 120.2 mm to (2.54, 69.0), turned to 180 degrees
- moved U$100 119.2 mm to (9.65, 38.7)
- moved U$218 119.0 mm to (2.54, 80.3), flipped to the top, turned to 0 degrees
- moved U$99 118.4 mm to (13.0, 38.5)
- moved U$98 118.0 mm to (16.0, 38.6)
- moved U$87 114.9 mm to (16.5, 29.2), turned to 0 degrees
- moved U$105 114.8 mm to (2.54, 45.6), flipped to the top, turned to 0 degrees
- moved U$93 114.4 mm to (26.7, 49.7)
- moved U$79 112.9 mm to (33.0, 49.7), turned to 270 degrees
- moved U$103 112.3 mm to (7.62, 45.1), flipped to the top, turned to 0 degrees
- moved U$102 112.1 mm to (10.9, 50.0), flipped to the top, turned to 0 degrees
- moved R65 110.2 mm to (21.0, 69.5), turned to 180 degrees
- moved U$80 108.5 mm to (30.5, 49.7), turned to 270 degrees
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Connections:
- removed net !FAN_EN10: R118.1, U21.11
- removed net !FAN_EN11: R129.1, U23.11
- removed net !FAN_EN12: R140.1, U25.11
- removed net !FAN_EN13: R151.1, U27.11
- removed net !FAN_EN14: R162.1, U29.11
- removed net !FAN_EN8: R96.1, U17.11
- removed net !FAN_EN9: R107.1, U19.11
- removed net !RST10: J63.5, R114.1, U21.4
- removed net !RST11: J69.5, R125.1, U23.4
- removed net !RST12: J75.5, R136.1, U25.4
- removed net !RST13: J81.5, R147.1, U27.4
- removed net !RST14: J87.5, R158.1, U29.4
- removed net !RST8: J51.5, R92.1, U17.4
- removed net !RST9: J57.5, R103.1, U19.4
- removed net 3.3V10: C52.1, J61.2, J62.2, J64.2, L11.1, Q31.1, Q32.1, R112.2, R116.2, U22.2, U22.3
- removed net 3.3V11: C57.1, J67.2, J68.2, J70.2, L12.1, Q34.1, Q35.1, R123.2, R127.2, U24.2, U24.3
- removed net 3.3V12: C62.1, J73.2, J74.2, J76.2, L13.1, Q37.1, Q38.1, R134.2, R138.2, U26.2, U26.3
- removed net 3.3V13: C67.1, J79.2, J80.2, J82.2, L14.1, Q40.1, Q41.1, R145.2, R149.2, U28.2, U28.3
- removed net 3.3V14: C72.1, J85.2, J86.2, J88.2, L15.1, Q43.1, Q44.1, R156.2, R160.2, U30.2, U30.3
- removed net 3.3V8: C42.1, J49.2, J50.2, J52.2, L9.1, Q25.1, Q26.1, R90.2, R94.2, U18.2, U18.3
- removed net 3.3V9: C47.1, J55.2, J56.2, J58.2, L10.1, Q28.1, Q29.1, R101.2, R105.2, U20.2, U20.3
- removed net 5V10: C53.1, D33.A, F11.2, J63.2, JP11.1, R113.2, R114.2, R117.2, U21.1, VR21.1, VR22.1
- removed net 5V11: C58.1, D36.A, F12.2, J69.2, JP12.1, R124.2, R125.2, R128.2, U23.1, VR23.1, VR24.1
- removed net 5V12: C63.1, D39.A, F13.2, J75.2, JP13.1, R135.2, R136.2, R139.2, U25.1, VR25.1, VR26.1
- removed net 5V13: C68.1, D42.A, F14.2, J81.2, JP14.1, R146.2, R147.2, R150.2, U27.1, VR27.1, VR28.1
- removed net 5V14: C73.1, D45.A, F15.2, J87.2, JP15.1, R157.2, R158.2, R161.2, U29.1, VR29.1, VR30.1
- removed net 5V8: C43.1, D27.A, F9.2, J51.2, JP9.1, R91.2, R92.2, R95.2, U17.1, VR17.1, VR18.1
- removed net 5V9: C48.1, D30.A, F10.2, J57.2, JP10.1, R102.2, R103.2, R106.2, U19.1, VR19.1, VR20.1
- removed net CIPO10: J63.1, U21.8
- removed net CIPO11: J69.1, U23.8
- removed net CIPO12: J75.1, U25.8
- removed net CIPO13: J81.1, U27.8
- removed net CIPO14: J87.1, U29.8
- removed net CIPO8: J51.1, U17.8
- removed net CIPO9: J57.1, U19.8
- removed net FAN_PWM10: D32.C, J65.4, U21.10
- removed net FAN_PWM11: D35.C, J71.4, U23.10
- removed net FAN_PWM12: D38.C, J77.4, U25.10
- removed net FAN_PWM13: D41.C, J83.4, U27.10
- removed net FAN_PWM14: D44.C, J89.4, U29.10
- removed net FAN_PWM8: D26.C, J53.4, U17.10
- removed net FAN_PWM9: D29.C, J59.4, U19.10
- removed net FAN_PWR10: J65.2, Q33.3
- removed net FAN_PWR11: J71.2, Q36.3
- removed net FAN_PWR12: J77.2, Q39.3
- removed net FAN_PWR13: J83.2, Q42.3
- removed net FAN_PWR14: J89.2, Q45.3
- removed net FAN_PWR8: J53.2, Q27.3
- removed net FAN_PWR9: J59.2, Q30.3
- removed net FAN_TACH10: D31.C, J65.3, R120.1, U21.6
- removed net FAN_TACH11: D34.C, J71.3, R131.1, U23.6
- removed net FAN_TACH12: D37.C, J77.3, R142.1, U25.6
- removed net FAN_TACH13: D40.C, J83.3, R153.1, U27.6
- removed net FAN_TACH14: D43.C, J89.3, R164.1, U29.6
- removed net FAN_TACH8: D25.C, J53.3, R98.1, U17.6
- removed net FAN_TACH9: D28.C, J59.3, R109.1, U19.6
- removed net GND10: C51.1, C52.2, C53.2, C54.1, C55.2, D31.A, D32.A, J61.1, J62.1, J63.6, J64.1, J65.1, J66.1, R115.1, R121.1, U21.14, U22.4, U22.8, VR21.3, VR22.3
- removed net GND11: C56.1, C57.2, C58.2, C59.1, C60.2, D34.A, D35.A, J67.1, J68.1, J69.6, J70.1, J71.1, J72.1, R126.1, R132.1, U23.14, U24.4, U24.8, VR23.3, VR24.3
- removed net GND12: C61.1, C62.2, C63.2, C64.1, C65.2, D37.A, D38.A, J73.1, J74.1, J75.6, J76.1, J77.1, J78.1, R137.1, R143.1, U25.14, U26.4, U26.8, VR25.3, VR26.3
- removed net GND13: C66.1, C67.2, C68.2, C69.1, C70.2, D40.A, D41.A, J79.1, J80.1, J81.6, J82.1, J83.1, J84.1, R148.1, R154.1, U27.14, U28.4, U28.8, VR27.3, VR28.3
- removed net GND14: C71.1, C72.2, C73.2, C74.1, C75.2, D43.A, D44.A, J85.1, J86.1, J87.6, J88.1, J89.1, J90.1, R159.1, R165.1, U29.14, U30.4, U30.8, VR29.3, VR30.3
- removed net GND8: C41.1, C42.2, C43.2, C44.1, C45.2, D25.A, D26.A, J49.1, J50.1, J51.6, J52.1, J53.1, J54.1, R93.1, R99.1, U17.14, U18.4, U18.8, VR17.3, VR18.3
- removed net GND9: C46.1, C47.2, C48.2, C49.1, C50.2, D28.A, D29.A, J55.1, J56.1, J57.6, J58.1, J59.1, J60.1, R104.1, R110.1, U19.14, U20.4, U20.8, VR19.3, VR20.3
- removed net HV_SCL10: J63.3, Q31.3, R113.1, U21.9
- removed net HV_SCL11: J69.3, Q34.3, R124.1, U23.9
- removed net HV_SCL12: J75.3, Q37.3, R135.1, U25.9
- removed net HV_SCL13: J81.3, Q40.3, R146.1, U27.9
- removed net HV_SCL14: J87.3, Q43.3, R157.1, U29.9
- removed net HV_SCL8: J51.3, Q25.3, R91.1, U17.9
- removed net HV_SCL9: J57.3, Q28.3, R102.1, U19.9
- removed net HV_SDA10: J63.4, Q32.3, R117.1, U21.7
- removed net HV_SDA11: J69.4, Q35.3, R128.1, U23.7
- removed net HV_SDA12: J75.4, Q38.3, R139.1, U25.7
- removed net HV_SDA13: J81.4, Q41.3, R150.1, U27.7
- removed net HV_SDA14: J87.4, Q44.3, R161.1, U29.7
- removed net HV_SDA8: J51.4, Q26.3, R95.1, U17.7
- removed net HV_SDA9: J57.4, Q29.3, R106.1, U19.7
- removed net KI_TRIM10: U21.13, VR22.2
- removed net KI_TRIM11: U23.13, VR24.2
- removed net KI_TRIM12: U25.13, VR26.2
- removed net KI_TRIM13: U27.13, VR28.2
- removed net KI_TRIM14: U29.13, VR30.2
- removed net KI_TRIM8: U17.13, VR18.2
- removed net KI_TRIM9: U19.13, VR20.2
- removed net KP_TRIM10: U21.12, VR21.2
- removed net KP_TRIM11: U23.12, VR23.2
- removed net KP_TRIM12: U25.12, VR25.2
- removed net KP_TRIM13: U27.12, VR27.2
- removed net KP_TRIM14: U29.12, VR29.2
- removed net KP_TRIM8: U17.12, VR17.2
- removed net KP_TRIM9: U19.12, VR19.2
- removed net N$100: L15.2, U30.1
- removed net N$101: C74.2, U29.3, Y15.1
- removed net N$102: C71.2, U29.2, Y15.3
- removed net N$103: Q45.1, R162.2, R163.1
- removed net N$104: C75.1, F15.1, R155.2, U30.7
- removed net N$105: D45.C, R165.2
- removed net N$20 (its old number): C15.1, F3.1, R23.2, U6.7
- removed net N$21 (its old number): D9.C, R33.2
- removed net N$22 (its old number): R34.1, R38.2, U8.5
- removed net N$29 (its old number): R45.1, R49.2, U10.5
- removed net N$40 (its old number): Q18.1, R63.2, R64.1
- removed net N$47 (its old number): Q21.1, R74.2, R75.1
- removed net N$48 (its old number): C35.1, F7.1, R67.2, U14.7
- removed net N$49 (its old number): D21.C, R77.2
- removed net N$56 (its old number): D24.C, R88.2
- removed net N$57 (its old number): R89.1, R93.2, U18.5
- removed net N$58 (its old number): L9.2, U18.1
- removed net N$65 (its old number): L10.2, U20.1
- removed net N$66 (its old number): C49.2, U19.3, Y10.1
- removed net N$67 (its old number): C46.2, U19.2, Y10.3
- removed net N$73: C54.2, U21.3, Y11.1
- removed net N$74: C51.2, U21.2, Y11.3
- removed net N$75: Q33.1, R118.2, R119.1
- removed net N$76: C55.1, F11.1, R111.2, U22.7
- removed net N$77: D33.C, R121.2
- removed net N$78: R122.1, R126.2, U24.5
- removed net N$79: L12.2, U24.1
- removed net N$80: C59.2, U23.3, Y12.1
- removed net N$81: C56.2, U23.2, Y12.3
- removed net N$82: Q36.1, R129.2, R130.1
- removed net N$83: C60.1, F12.1, R122.2, U24.7
- removed net N$84: D36.C, R132.2
- removed net N$85: R133.1, R137.2, U26.5
- removed net N$86: L13.2, U26.1
- removed net N$87: C64.2, U25.3, Y13.1
- removed net N$88: C61.2, U25.2, Y13.3
- removed net N$89: Q39.1, R140.2, R141.1
- removed net N$90: C65.1, F13.1, R133.2, U26.7
- removed net N$91: D39.C, R143.2
- removed net N$92: R144.1, R148.2, U28.5
- removed net N$93: L14.2, U28.1
- removed net N$94: C69.2, U27.3, Y14.1
- removed net N$95: C66.2, U27.2, Y14.3
- removed net N$96: Q42.1, R151.2, R152.1
- removed net N$97: C70.1, F14.1, R144.2, U28.7
- removed net N$98: D42.C, R154.2
- removed net N$99: R155.1, R159.2, U30.5
- removed net SCL10: J61.4, J62.4, J64.4, Q31.2, R112.1
- removed net SCL11: J67.4, J68.4, J70.4, Q34.2, R123.1
- removed net SCL12: J73.4, J74.4, J76.4, Q37.2, R134.1
- removed net SCL13: J79.4, J80.4, J82.4, Q40.2, R145.1
- removed net SCL14: J85.4, J86.4, J88.4, Q43.2, R156.1
- removed net SCL8: J49.4, J50.4, J52.4, Q25.2, R90.1
- removed net SCL9: J55.4, J56.4, J58.4, Q28.2, R101.1
- removed net SDA10: J61.3, J62.3, J64.3, Q32.2, R116.1
- removed net SDA11: J67.3, J68.3, J70.3, Q35.2, R127.1
- removed net SDA12: J73.3, J74.3, J76.3, Q38.2, R138.1
- removed net SDA13: J79.3, J80.3, J82.3, Q41.2, R149.1
- removed net SDA14: J85.3, J86.3, J88.3, Q44.2, R160.1
- removed net SDA8: J49.3, J50.3, J52.3, Q26.2, R94.1
- removed net SDA9: J55.3, J56.3, J58.3, Q29.2, R105.1
- removed net VCC_10: J60.2, JP10.2, Q30.2, R108.2, R109.2
- removed net VCC_11: J66.2, JP11.2, Q33.2, R119.2, R120.2
- removed net VCC_12: J72.2, JP12.2, Q36.2, R130.2, R131.2
- removed net VCC_13: J78.2, JP13.2, Q39.2, R141.2, R142.2
- removed net VCC_14: J84.2, JP14.2, Q42.2, R152.2, R153.2
- removed net VCC_15: J90.2, JP15.2, Q45.2, R163.2, R164.2
- removed net VCC_9: J54.2, JP9.2, Q27.2, R97.2, R98.2
- new net N$16: Q8.2, Q8.5, Q8.6, R12.2
- new net N$17: Q10.3, Q9.1, R25.2
- new net N$18: Q10.2, Q10.5, Q10.6, R26.2
- new net N$23: Q13.1, R34.2, R35.1
- new net N$24: C15.1, F3.1, R27.2, U6.7
- new net N$25: D9.C, R37.2
- new net N$32: Q18.1, R47.2, R48.1
- new net N$37: R53.1, R57.2, U10.5
- new net N$44: Q24.1, Q25.3, R64.2
- new net N$45: Q25.2, Q25.5, Q25.6, R65.2
- new net N$46: R66.1, R70.2, U12.5
- new net N$51: C30.1, F6.1, R66.2, U12.7
- new net N$52: D18.C, R76.2
- new net N$53: Q29.1, Q30.3, R77.2
- net !FAN_EN1: now also R21.1; no longer R19.1
- net !FAN_EN2: now also R34.1; no longer R30.1
- net !FAN_EN3: now also R47.1; no longer R41.1
- net !FAN_EN4: now also R60.1; no longer R52.1
- net !FAN_EN5: now also R73.1; no longer R63.1
- net !FAN_EN6: now also R86.1; no longer R74.1
- net !FAN_EN7: now also R99.1; no longer R85.1
- net !RST1: now also R17.1; no longer R15.1
- net !RST2: now also R30.1; no longer R26.1
- net !RST3: now also R43.1; no longer R37.1
- net !RST4: now also R56.1; no longer R48.1
- net !RST5: now also R69.1; no longer R59.1
- net !RST6: now also R82.1; no longer R70.1
- net !RST7: now also R95.1; no longer R81.1
- net 3.3V1: now also R15.2, R19.2; no longer R12.2, R17.2
- net 3.3V2: now also Q11.1, Q12.1, R32.2; no longer Q7.1, Q8.1, R24.2
- net 3.3V3: now also Q16.1, Q17.1, R41.2, R45.2; no longer Q10.1, Q11.1, R35.2, R39.2
- net 3.3V4: now also Q21.1, Q22.1, R54.2, R58.2; no longer Q13.1, Q14.1, R46.2, R50.2
- net 3.3V5: now also Q26.1, Q27.1, R67.2, R71.2; no longer Q16.1, Q17.1, R57.2, R61.2
- net 3.3V6: now also Q31.1, Q32.1, R80.2, R84.2; no longer Q19.1, Q20.1, R68.2, R72.2
- net 3.3V7: now also Q36.1, Q37.1, R93.2, R97.2; no longer Q22.1, Q23.1, R79.2, R83.2
- net 5V: now also Q7.3, Q8.1; no longer JP1.1
- net 5V1: now also Q10.1, Q9.3, R16.2, R17.2, R20.2; no longer JP2.1, R14.2, R15.2, R18.2
- net 5V2: now also Q14.3, Q15.1, R30.2, R33.2; no longer JP3.1, R25.2, R26.2
- net 5V3: now also Q19.3, Q20.1, R42.2, R43.2, R46.2; no longer JP4.1, R36.2, R37.2, R40.2
- net 5V4: now also Q24.3, Q25.1, R55.2, R56.2, R59.2; no longer JP5.1, R47.2, R48.2, R51.2
- net 5V5: now also Q29.3, Q30.1, R68.2, R69.2, R72.2; no longer JP6.1, R58.2, R59.2, R62.2
- net 5V6: now also Q34.3, Q35.1, R81.2, R82.2, R85.2; no longer JP7.1, R69.2, R70.2, R73.2
- net 5V7: now also Q39.3, Q40.1, R94.2, R95.2, R98.2; no longer JP8.1, R80.2, R81.2, R84.2
- net FAN_PWR2: now also Q13.3; no longer Q9.3
- net FAN_PWR3: now also Q18.3; no longer Q12.3
- net FAN_PWR4: now also Q23.3; no longer Q15.3
- net FAN_PWR5: now also Q28.3; no longer Q18.3
- net FAN_PWR6: now also Q33.3; no longer Q21.3
- net FAN_PWR7: now also Q38.3; no longer Q24.3
- net FAN_TACH1: now also R23.1; no longer R21.1
- net FAN_TACH2: now also R36.1; no longer R32.1
- net FAN_TACH3: now also R49.1; no longer R43.1
- net FAN_TACH4: now also R62.1; no longer R54.1
- net FAN_TACH5: now also R75.1; no longer R65.1
- net FAN_TACH6: now also R88.1; no longer R76.1
- net FAN_TACH7: now also R101.1; no longer R87.1
- net GND: now also R10.1, R12.1
- net GND1: now also R18.1, R24.1, R25.1, R26.1; no longer R16.1, R22.1
- net GND2: now also R31.1, R37.1, R38.1, R39.1; no longer R27.1, R33.1
- net GND3: now also R50.1, R51.1, R52.1; no longer R38.1
- net GND4: now also R57.1, R63.1, R64.1, R65.1; no longer R49.1, R55.1
- net GND5: now also R70.1, R76.1, R77.1, R78.1; no longer R60.1, R66.1
- net GND6: now also R83.1, R89.1, R90.1, R91.1; no longer R71.1, R77.1
- net GND7: now also R102.1, R103.1, R104.1, R96.1; no longer R82.1, R88.1
- net HV_SCL1: now also R16.1; no longer R14.1
- net HV_SCL2: now also Q11.3, R29.1; no longer Q7.3, R25.1
- net HV_SCL3: now also Q16.3, R42.1; no longer Q10.3, R36.1
- net HV_SCL4: now also Q21.3, R55.1; no longer Q13.3, R47.1
- net HV_SCL5: now also Q26.3, R68.1; no longer Q16.3, R58.1
- net HV_SCL6: now also Q31.3, R81.1; no longer Q19.3, R69.1
- net HV_SCL7: now also Q36.3, R94.1; no longer Q22.3, R80.1
- net HV_SDA1: now also R20.1; no longer R18.1
- net HV_SDA2: now also Q12.3, R33.1; no longer Q8.3, R29.1
- net HV_SDA3: now also Q17.3, R46.1; no longer Q11.3, R40.1
- net HV_SDA4: now also Q22.3, R59.1; no longer Q14.3, R51.1
- net HV_SDA5: now also Q27.3, R72.1; no longer Q17.3, R62.1
- net HV_SDA6: now also Q32.3, R85.1; no longer Q20.3, R73.1
- net HV_SDA7: now also Q37.3, R98.1; no longer Q23.3, R84.1
- net N$12: now also R21.2, R22.1; no longer R19.2, R20.1
- net N$13: now also R14.2; no longer R10.2
- net N$14: now also R24.2; no longer R22.2
- net N$15: now also Q7.1, Q8.3, R10.2; no longer R23.1, R27.2, U6.5
- net N$19: now also R27.1, R31.2, U6.5; no longer Q9.1, R30.2, R31.1
- net N$26: now also Q14.1, Q15.3, R38.2; no longer Q12.1, R41.2, R42.1
- net N$27: now also Q15.2, Q15.5, Q15.6, R39.2; no longer C20.1, F4.1, R34.2, U8.7
- net N$28: now also R40.1, U8.5; no longer D12.C
- net N$33: now also C20.1, F4.1, R40.2, U8.7; no longer Q15.1, R52.2, R53.1
- net N$34: now also D12.C, R50.2; no longer C25.1, F5.1, R45.2, U10.7
- net N$35: now also Q19.1, Q20.3, R51.2; no longer D15.C, R55.2
- net N$36: now also Q20.2, Q20.5, Q20.6, R52.2; no longer R56.1, R60.2, U12.5
- net N$41: now also Q23.1, R60.2, R61.1; no longer C30.1, F6.1, R56.2, U12.7
- net N$42: now also C25.1, F5.1, R53.2, U10.7; no longer D18.C, R66.2
- net N$43: now also D15.C, R63.2; no longer R67.1, R71.2, U14.5
- net N$50: now also Q28.1, R73.2, R74.1; no longer R78.1, R82.2, U16.5
- net N$54: now also Q30.2, Q30.5, Q30.6, R78.2; no longer Q24.1, R85.2, R86.1
- net N$55: now also R79.1, R83.2, U14.5; no longer C40.1, F8.1, R78.2, U16.7
- net N$59: now also Q33.1, R86.2, R87.1; no longer C44.2, U17.3, Y9.1
- net N$60: now also C35.1, F7.1, R79.2, U14.7; no longer C41.2, U17.2, Y9.3
- net N$61: now also D21.C, R89.2; no longer Q27.1, R96.2, R97.1
- net N$62: now also Q34.1, Q35.3, R90.2; no longer C45.1, F9.1, R89.2, U18.7
- net N$63: now also Q35.2, Q35.5, Q35.6, R91.2; no longer D27.C, R99.2
- net N$64: now also R92.1, R96.2, U16.5; no longer R100.1, R104.2, U20.5
- net N$68: now also Q38.1, R100.1, R99.2; no longer Q30.1, R107.2, R108.1
- net N$69: now also C40.1, F8.1, R92.2, U16.7; no longer C50.1, F10.1, R100.2, U20.7
- net N$70: now also D24.C, R102.2; no longer D30.C, R110.2
- net N$71: now also Q39.1, Q40.3, R103.2; no longer R111.1, R115.2, U22.5
- net N$72: now also Q40.2, Q40.5, Q40.6, R104.2; no longer L11.2, U22.1
- net N$8: now also R14.1, R18.2; no longer R10.1, R16.2
- net SCL1: now also R15.1; no longer R12.1
- net SCL2: now also Q11.2, R28.1; no longer Q7.2, R24.1
- net SCL3: now also Q16.2, R41.1; no longer Q10.2, R35.1
- net SCL4: now also Q21.2, R54.1; no longer Q13.2, R46.1
- net SCL5: now also Q26.2, R67.1; no longer Q16.2, R57.1
- net SCL6: now also Q31.2, R80.1; no longer Q19.2, R68.1
- net SCL7: now also Q36.2, R93.1; no longer Q22.2, R79.1
- net SDA1: now also R19.1; no longer R17.1
- net SDA2: now also Q12.2, R32.1; no longer Q8.2, R28.1
- net SDA3: now also Q17.2, R45.1; no longer Q11.2, R39.1
- net SDA4: now also Q22.2, R58.1; no longer Q14.2, R50.1
- net SDA5: now also Q27.2, R71.1; no longer Q17.2, R61.1
- net SDA6: now also Q32.2, R84.1; no longer Q20.2, R72.1
- net SDA7: now also Q37.2, R97.1; no longer Q23.2, R83.1
- net VCC_1: now also Q10.4, Q9.2, R22.2, R23.2; no longer JP2.2, R20.2, R21.2
- net VCC_2: now also Q7.2, Q8.4; no longer JP1.2
- net VCC_3: now also Q13.2, Q14.2, Q15.4, R35.2, R36.2; no longer JP3.2, Q9.2, R31.2, R32.2
- net VCC_4: now also Q18.2, Q19.2, Q20.4, R48.2, R49.2; no longer JP4.2, Q12.2, R42.2, R43.2
- net VCC_5: now also Q23.2, Q24.2, Q25.4, R61.2, R62.2; no longer JP5.2, Q15.2, R53.2, R54.2
- net VCC_6: now also Q28.2, Q29.2, Q30.4, R74.2, R75.2; no longer JP6.2, Q18.2, R64.2, R65.2
- net VCC_7: now also Q33.2, Q34.2, Q35.4, R87.2, R88.2; no longer JP7.2, Q21.2, R75.2, R76.2
- net VCC_8: now also Q38.2, Q39.2, Q40.4, R100.2, R101.2; no longer JP8.2, Q24.2, R86.2, R87.2
Routing:
- net 5V14: track 79.0 -> 0.00 mm, vias 5 -> 0
- net 5V11: track 79.0 -> 0.00 mm, vias 5 -> 0
- net 5V9: track 79.0 -> 0.00 mm, vias 5 -> 0
- net 5V13: track 79.0 -> 0.00 mm, vias 5 -> 0
- net 5V12: track 79.0 -> 0.00 mm, vias 5 -> 0
- net 5V10: track 79.0 -> 0.00 mm, vias 5 -> 0
- net 5V8: track 79.0 -> 0.00 mm, vias 5 -> 0
- net 3.3V9: track 69.7 -> 0.00 mm, vias 5 -> 0
- net 3.3V8: track 69.7 -> 0.00 mm, vias 5 -> 0
- net 3.3V11: track 69.7 -> 0.00 mm, vias 5 -> 0
- net 3.3V14: track 69.7 -> 0.00 mm, vias 5 -> 0
- net 3.3V13: track 69.7 -> 0.00 mm, vias 5 -> 0
- net 3.3V12: track 69.7 -> 0.00 mm, vias 5 -> 0
- net 3.3V10: track 69.7 -> 0.00 mm, vias 5 -> 0
- net SDA8: track 63.0 -> 0.00 mm, vias 3 -> 0
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- removed copper zone on layer 1, net GND10
- removed copper zone on layer 16, net GND10
- removed copper zone on layer 1, net GND11
- removed copper zone on layer 16, net GND11
- removed copper zone on layer 1, net GND12
- removed copper zone on layer 16, net GND12
- removed copper zone on layer 1, net GND13
- removed copper zone on layer 16, net GND13
- removed copper zone on layer 1, net GND14
- removed copper zone on layer 16, net GND14
- removed copper zone on layer 1, net GND8
- removed copper zone on layer 16, net GND8
- removed copper zone on layer 1, net GND9
- removed copper zone on layer 16, net GND9
Other:
- board size 158.2 x 143.3 mm -> 112 x 117.3 mm
- board text added: "x02"
- board text removed: "x01"
